File: TouCAN.kicad_sch (KiCad schematic)
At the start: 99 parts, among them J1 m12_M_CAN_90, J10 Conn_01x04, J11 Conn_01x03, J2 USB4105GFA060, J3 DTF13-3P, J4 m12_M_CAN_90, J5 Conn_01x03, J7 DTF13-3P, J8 Conn_01x04, J9 USB_A_Stacked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

Commit message: major changes removed m12 and changed layout
Parts:
- removed C1, C10, C11, C15, C17, C18, C20, C22, C24, C26, C37, C38, C40, C41: 100nf, Capacitor_SMD:C_0603_1608Metric, symbol Device:C_Small
- removed C12, C16, C21, C25: 10nf, Capacitor_SMD:C_0603_1608Metric, symbol Device:C_Small
- removed C13, C14, C19, C23, C7, C8, C9: 10uf, Capacitor_SMD:C_0603_1608Metric, symbol Device:C_Small
- removed C2, C27, C28, C29, C3, C30, C31, C4, C5, C6: 22uf, Capacitor_SMD:C_0603_1608Metric, symbol Device:C_Small
- removed C32, C33, C36, C39: 100nF, Capacitor_SMD:C_0402_1005Metric, symbol Device:C_Small
- removed C34, C35: 18pF, Capacitor_SMD:C_0402_1005Metric, symbol Device:C_Small
- removed D1, D2: ESDA6V1L, Package_TO_SOT_SMD:SOT-23-3, symbol Ethan_library:ESDA6V1L
- removed D3: PRTR5V0U2X, Package_TO_SOT_SMD:SOT-143, symbol Power_Protection:PRTR5V0U2X
- removed D4, D7: green, LED_SMD:LED_0603_1608Metric, symbol Device:LED_Small
- removed D5, D6: blue, LED_SMD:LED_0603_1608Metric, symbol Device:LED_Small
- removed D8: red, LED_SMD:LED_0603_1608Metric, symbol Device:LED_Small
- removed J1, J4: m12_M_CAN_90, Ethan_footprints:M12A-05PMMR-EE0001, symbol Ethan_library:m12_M_90
- removed J10, J8: Conn_01x04, Connector_PinSocket_2.54mm:PinSocket_1x04_P2.54mm_Vertical, symbol Connector_Generic:Conn_01x04
- removed J11, J5: Conn_01x03, Connector_PinHeader_2.54mm:PinHeader_1x03_P2.54mm_Vertical, symbol Connector_Generic:Conn_01x03
- removed J2: USB4105GFA060, Ethan_footprints:GCT_USB4105GFA060, symbol Ethan_library:USB4105GFA060
- removed J3, J7: DTF13-3P, Ethan_footprints:DTF13-3P, symbol Ethan_library:DTF13-3P
- removed J9: USB_A_Stacked, Connector_USB:USB_A_CUI_UJ2-ADH-TH_Horizontal_Stacked, symbol Connector:USB_A_Stacked
- removed Q1, Q3: PMOS, Ethan_footprints:PMV48XP, symbol Simulation_SPICE:PMOS
- removed R1, R6: 10r, Resistor_SMD:R_0603_1608Metric, symbol Device:R_Small
- removed R10, R11, R7, R8, R9: 1k, Resistor_SMD:R_0603_1608Metric, symbol Device:R_Small
- removed R12: 12k, Resistor_SMD:R_0402_1005Metric, symbol Device:R_Small
- removed R13, R14, R15, R21, R22: 100k, Resistor_SMD:R_0402_1005Metric, symbol Device:R_Small
- removed R16, R17, R18, R19: 10k, Resistor_SMD:R_0603_1608Metric, symbol Device:R_Small
- removed R2, R5: 120r, Resistor_SMD:R_0603_1608Metric, symbol Device:R_Small
- removed R20: 1M, Resistor_SMD:R_0603_1608Metric, symbol Device:R_Small
- removed R23, R24: 0R, Resistor_SMD:R_0402_1005Metric, symbol Device:R_Small
- removed R25, R26: 100k, Resistor_SMD:R_0603_1608Metric, symbol Device:R_Small
- removed R3, R4: 5.1k, Resistor_SMD:R_0603_1608Metric, symbol Device:R_Small
- removed SW1, SW3: OS102011MA1QN1, Ethan_footprints:OS102011MA1QN1, symbol Ethan_library:OS102011MA1QN1
- removed TP1, TP2, TP3: testpad, TestPoint:TestPoint_Pad_D1.0mm, symbol Connector:TestPoint
- removed U1, U5: STM32G431C6Tx, Package_QFP:LQFP-48_7x7mm_P0.5mm, symbol MCU_ST_STM32G4:STM32G431C6Tx
- removed U2: USB2514B_Bi, Package_DFN_QFN:QFN-36-1EP_6x6mm_P0.5mm_EP3.7x3.7mm, symbol Ethan_library:USB2514B_Bi
- removed U3, U6: ADM3053, Package_SO:SOIC-20W_7.5x12.8mm_P1.27mm, symbol Interface_CAN_LIN:ADM3053
- removed U7: RS3236-3.3YF5, Package_TO_SOT_SMD:SOT-23-5, symbol Ethan_library:RS3236-3.3YF5
- removed Y1: 24mhz, Crystal:Crystal_SMD_3225-4Pin_3.2x2.5mm, symbol Device:Crystal_GND24_Small
Connections:
- no-connect marks 14 -> 0
Other:
- added sheet Brains (Brains.kicad_sch)
- added sheet Brains2 (Brains2.kicad_sch)
- added sheet CAN (CAN.kicad_sch)
- added sheet CAN2 (CAN2.kicad_sch)
- added sheet Power (untitled.kicad_sch)
- added sheet hub (hub.kicad_sch)
- note removed: "BOOT"
- note removed: "CAN"
- note removed: "PRGM"
- note removed: "Power On Delay"
